File: Hardware/Temperature Sensor Board/Temperature Senor Board V2 (2).kicad_pcb (KiCad board)
At the start: 2 copper layers, 41.9 x 26.3 mm, 3 parts

Commit message: Gerber File  Changed
Parts:
- removed E2: TEMP_SENSOR_1, 1734723-1_RJ11
- removed R2: , R0805
- added 4.7k: R, AutoLoadbankFootprint:R0805, F.Cu at (135.9, 88.7)
- added J2: 6P6C, AutoLoadbankFootprint:1734723-1_RJ11, F.Cu at (161.0, 87.8)
- U$1: value DS18B -> Temperature Sensor 1; footprint TO92 -> AutoLoadbankFootprint:TO92-3
- moved U$1 15.2 mm to (123.4, 88.3)
Connections:
- U$1 pad 1: GND -> /GND
- U$1 pad 2: DQ -> /DQ
- U$1 pad 3: VDD -> /VDD
Routing:
- net /VDD: track 0.00 -> 47.4 mm
- net GND: track 46.8 -> 0.00 mm
- net /DQ: track 0.00 -> 38.1 mm
- net VDD: track 30.0 -> 0.00 mm
- net DQ: track 23.5 -> 0.00 mm
- net /GND: vias 0 -> 8
- added copper zone on B.Cu, net /GND
- added copper zone on F.Cu, net /GND
Other:
- board size 41.9 x 26.3 mm -> 55.9 x 23.1 mm
- board text added: "TEMP_SENSOR_1"

Commit message: edit
Parts:
- moved 4.7k 2.30 mm to (134.1, 90.2)
- moved U$1 1.72 mm to (124.9, 89.2)
Routing:
- net /VDD: track 47.4 -> 43.1 mm
- net /DQ: track 38.1 -> 35.9 mm
Other:
- board text added: "DQ"
- board text added: "VDD"
Changed lines of the file:
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@@
       (drillshape 0)
       (scaleselection 1)
-      (outputdirectory "New(3) Gerber File/")
+      (outputdirectory "Temp_Sens1_v2_gerber")
     )
   )
@@
   )
   (footprint "AutoLoadbankFootprint:TO92-3" (layer "F.Cu")
-    (at 123.443979 88.265031 -90)
+    (at 124.8664 89.2302 -90)
     (descr "<b>TO 92</b>")
     (property "Sheetfile" "Temperature Senor Board V2 (2).kicad_sch")
@@
         (effects (font (size 1.143 1.143) (thickness 0.127)) (justify right bottom))
     )
-    (fp_text user "2" (at 1.142969 -3.683021) (layer "F.SilkS")
+    (fp_text user "2" (at -0.2794 -3.7846) (layer "F.SilkS")
         (effects (font (size 1.143 1.143) (thickness 0.127)) (justify right bottom))
     )
@@
   )
   (footprint "AutoLoadbankFootprint:R0805" (layer "F.Cu")
-    (at 135.89 88.712 -90)
+    (at 134.112 90.17 -90)
     (descr "<b>RESISTOR</b><p>")
     (property "Sheetfile" "Temperature Senor Board V2 (2).kicad_sch")
@@
     (property "ki_description" "Resistor")
     (property "ki_keywords" "R res resistor")
-    (fp_text reference "4.7k" (at -2.987 1.524) (layer "F.SilkS")
+    (fp_text reference "4.7k" (at -2.2352 1.6002) (layer "F.SilkS")
         (effects (font (size 1.1684 1.1684) (thickness 0.1016)) (justify left bottom))
     )
@@
   (gr_rect (start 119.761 76.327) (end 175.641 99.441)
     (stroke (width 0.05) (type default)) (fill none) (layer "Edge.Cuts"))
-  (gr_text "TEMP_SENSOR_1\n" (at 156.976 80.222) (layer "F.SilkS")
+  (gr_text "VDD" (at 164.6936 88.9762) (layer "B.SilkS")
+    (effects (font (size 1 1) (thickness 0.1)) (justify left bottom mirror))
+  )
+  (gr_text "DQ" (at 164.1094 91.821) (layer "B.SilkS")
+    (effects (font (size 1 1) (thickness 0.1)) (justify left bottom mirror))
+  )
+  (gr_text "TEMP_SENSOR_1\n" (at 156.9466 79.9592) (layer "F.SilkS")
     (effects (font (size 1.143 1.143) (thickness 0.127)) (justify left bottom))
   )
-  (via (at 139.192 84.201) (size 0.6) (drill 0.3) (layers "F.Cu" "B.Cu") (free) (net 1))
-  (via (at 145.161 84.201) (size 0.6) (drill 0.3) (layers "F.Cu" "B.Cu") (free) (net 1))
-  (via (at 151.257 90.424) (size 0.6) (drill 0.3) (layers "F.Cu" "B.Cu") (free) (net 1))
+  (via (at 139.192 86.36) (size 0.6) (drill 0.3) (layers "F.Cu" "B.Cu") (free) (net 1))
+  (via (at 145.161 86.36) (size 0.6) (drill 0.3) (layers "F.Cu" "B.Cu") (free) (net 1))
+  (via (at 151.13 90.424) (size 0.6) (drill 0.3) (layers "F.Cu" "B.Cu") (free) (net 1))
   (via (at 139.192 90.424) (size 0.6) (drill 0.3) (layers "F.Cu" "B.Cu") (free) (net 1))
-  (via (at 151.257 84.201) (size 0.6) (drill 0.3) (layers "F.Cu" "B.Cu") (free) (net 1))
-  (via (at 130.175 91.567) (size 0.6) (drill 0.3) (layers "F.Cu" "B.Cu") (free) (net 1))
+  (via (at 151.13 86.36) (size 0.6) (drill 0.3) (layers "F.Cu" "B.Cu") (free) (net 1))
+  (via (at 130.4798 90.2208) (size 0.6) (drill 0.3) (layers "F.Cu" "B.Cu") (free) (net 1))
   (via (at 130.429 86.233) (size 0.6) (drill 0.3) (layers "F.Cu" "B.Cu") (free) (net 1))
   (via (at 145.161 90.424) (size 0.6) (drill 0.3) (layers "F.Cu" "B.Cu") (free) (net 1))
-  (segment (start 135.89 87.762) (end 125.85201 87.762) (width 0.2) (layer "F.Cu") (net 2))
-  (segment (start 161.036 90.495683) (end 159.298717 88.7584) (width 0.2) (layer "F.Cu") (net 2))
+  (segment (start 159.760317 89.22) (end 134.112 89.22) (width 0.2) (layer "F.Cu") (net 2))
   (segment (start 161.036 91.562) (end 161.036 90.495683) (width 0.2) (layer "F.Cu") (net 2))
-  (segment (start 159.298717 88.7584) (end 136.8864 88.7584) (width 0.2) (layer "F.Cu") (net 2))
-  (segment (start 136.8864 88.7584) (end 135.89 87.762) (width 0.2) (layer "F.Cu") (net 2))
-  (segment (start 125.85201 87.762) (end 125.348979 88.265031) (width 0.2) (layer "F.Cu") (net 2))
-  (segment (start 161.036 89.022) (end 163.195 91.181) (width 0.2) (layer "F.Cu") (net 3))
-  (segment (start 123.570948 89.662) (end 123.443979 89.535031) (width 0.2) (layer "F.Cu") (net 3))
-  (segment (start 163.195 91.181) (end 163.195 93.599) (width 0.2) (layer "F.Cu") (net 3))
-  (segment (start 135.89 89.662) (end 123.570948 89.662) (width 0.2) (layer "F.Cu") (net 3))
-  (segment (start 140.462 94.234) (end 135.89 89.662) (width 0.2) (layer "F.Cu") (net 3))
-  (segment (start 163.195 93.599) (end 162.56 94.234) (width 0.2) (layer "F.Cu") (net 3))
-  (segment (start 162.56 94.234) (end 140.462 94.234) (width 0.2) (layer "F.Cu") (net 3))
+  (segment (start 134.112 89.22) (end 126.7816 89.22) (width 0.2) (layer "F.Cu") (net 2))
+  (segment (start 126.7816 89.22) (end 126.7714 89.2302) (width 0.2) (layer "F.Cu") (net 2))
+  (segment (start 161.036 90.495683) (end 159.760317 89.22) (width 0.2) (layer "F.Cu") (net 2))
+  (segment (start 162.56 90.546) (end 162.56 91.948) (width 0.2) (layer "F.Cu") (net 3))
+  (segment (start 125.4862 91.12) (end 124.8664 90.5002) (width 0.2) (layer "F.Cu") (net 3))
+  (segment (start 161.036 89.022) (end 162.56 90.546) (width 0.2) (layer "F.Cu") (net 3))
+  (segment (start 162.56 91.948) (end 161.036 93.472) (width 0.2) (layer "F.Cu") (net 3))
+  (segment (start 161.036 93.472) (end 136.464 93.472) (width 0.2) (layer "F.Cu") (net 3))
+  (segment (start 136.464 93.472) (end 134.112 91.12) (width 0.2) (layer "F.Cu") (net 3))
+  (segment (start 134.112 91.12) (end 125.4862 91.12) (width 0.2) (layer "F.Cu") (net 3))
   (zone (net 1) (net_name "/GND") (layer "F.Cu") (hatch edge 0.5)
     (priority 1)
