File: Hardware/Temperature Sensor Board/Temperature Sensor Board 2/Temperature Sensor Board 2.kicad_pcb (KiCad board)
At the start: 2 copper layers, 41.3 x 19.9 mm, 3 parts, among them J1 6P6C

Commit message: complete gerber for temp sensors
Other:
- board text added: "DQ"
- board text added: "VDD"
Changed lines of the file:
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@@
       (plot_on_all_layers_selection 0x0000000_00000000)
       (disableapertmacros false)
-      (usegerberextensions false)
-      (usegerberattributes true)
-      (usegerberadvancedattributes true)
-      (creategerberjobfile true)
+      (usegerberextensions true)
+      (usegerberattributes false)
+      (usegerberadvancedattributes false)
+      (creategerberjobfile false)
       (dashed_line_dash_ratio 12.000000)
       (dashed_line_gap_ratio 3.000000)
@@
       (psa4output false)
       (plotreference true)
-      (plotvalue true)
+      (plotvalue false)
       (plotinvisibletext false)
       (sketchpadsonfab false)
-      (subtractmaskfromsilk false)
+      (subtractmaskfromsilk true)
       (outputformat 1)
       (mirror false)
       (drillshape 0)
       (scaleselection 1)
-      (outputdirectory "../../../Documents/GitHub/AutomatedLoadBank/Hardware/Temperature Sensor Board/Temperature Sensor Board 2/Gerber Files for Temp Sensor 2/")
+      (outputdirectory "temp_sens2_gerber/")
     )
   )
@@
   (gr_rect (start 109.687354 84.160354) (end 151.003 104.013)
     (stroke (width 0.1) (type default)) (fill none) (layer "Edge.Cuts"))
+  (gr_text "VDD" (at 140.1572 96.3422) (layer "B.SilkS")
+    (effects (font (size 1 1) (thickness 0.1)) (justify left bottom mirror))
+  )
+  (gr_text "DQ" (at 139.4206 98.8568) (layer "B.SilkS")
+    (effects (font (size 1 1) (thickness 0.1)) (justify left bottom mirror))
+  )
   (gr_text "TEMP_SENSOR_2" (at 147.279354 86.192354) (layer "F.SilkS")
     (effects (font (size 1.143 1.143) (thickness 0.127)) (justify right bottom))
