File: Hardware/Voltage Regulator Board/voltage-regulator/voltage-regulator.kicad_sch (KiCad schematic)
At the start: 0 parts

Commit message: sch capture
Parts:
- added J1: Conn_01x08_Socket, Connector_Phoenix_MSTB:PhoenixContact_MSTBA_2,5_8-G-5,08_1x08_P5.08mm_Horizontal, symbol Connector:Conn_01x08_Socket
Other:
- note added: "Board Edge Connector"
Changed lines of the file:
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@@
 (kicad_sch (version 20230121) (generator eeschema)
   (paper "A4")
+  (rectangle (start 55.88 16.51) (end 55.88 16.51)
+    (stroke (width 0) (type default))
+    (fill (type none))
+  )
+  (rectangle (start 17.78 16.51) (end 113.03 81.28)
+    (stroke (width 1) (type dash))
+    (fill (type none))
+  )
+  (text "Board Edge Connector" (at 31.75 25.4 0)
+    (effects (font (size 3 3) (thickness 0.6) bold) (justify left bottom))
+  )
+  (symbol (lib_id "Connector:Conn_01x08_Socket") (at 53.34 46.99 0) (unit 1)
+    (in_bom yes) (on_board yes) (dnp no)
+    (property "Reference" "J1" (at 44.45 48.26 0)
+      (effects (font (size 1.27 1.27)) (justify left))
+    )
+    (property "Value" "Conn_01x08_Socket" (at 27.94 50.8 0)
+      (effects (font (size 1.27 1.27)) (justify left))
+    )
+    (property "Footprint" "Connector_Phoenix_MSTB:PhoenixContact_MSTBA_2,5_8-G-5,08_1x08_P5.08mm_Horizontal" (at 53.34 46.99 0)
+      (effects (font (size 1.27 1.27)) hide)
+    )
+    (property "Datasheet" "~" (at 53.34 46.99 0)
+      (effects (font (size 1.27 1.27)) hide)
+    )
+    (pin "1")
+    (pin "2")
+    (pin "3")
+    (pin "4")
+    (pin "5")
+    (pin "6")
+    (pin "7")
+    (pin "8")
+    (instances
+      (project "voltage-regulator"
+        (path "/14e40bb6-60ec-4249-a8f7-92b65d5cdd04"
+          (reference "J1") (unit 1)
+        )
+      )
+    )
+  )
   (sheet_instances
     (path "/" (page "1"))

Commit message: sch capture 2
Parts:
- removed J1: Conn_01x08_Socket, Connector_Phoenix_MSTB:PhoenixContact_MSTBA_2,5_8-G-5,08_1x08_P5.08mm_Horizontal, symbol Connector:Conn_01x08_Socket
- added C1, C4: 0.1uF, Capacitor_SMD:C_0805_2012Metric, symbol Device:C
- added C10, C5, C6, C7, C8, C9: C, symbol Device:C
- added C11: C_Polarized, symbol Device:C_Polarized
- added C2, C3: 100uF, Capacitor_THT:CP_Radial_D8.0mm_P3.50mm, symbol Device:C_Polarized
- added CR1: L4978, DIP-8_STM, symbol 2024-01-04_22-26-55:L4978
- added D1, D2: 1N5822, Diode_THT:D_DO-201AD_P15.24mm_Horizontal, symbol Device:D
- added F1, F2: 5A, Fuse:Fuseholder_Blade_Mini_Keystone_3568, symbol Device:Fuse
- added HS1: Heatsink_Pad_2Pin, Heatsink:Heatsink_Fischer_SK129-STS_42x25mm_2xDrill2.5mm, symbol Mechanical:Heatsink_Pad_2Pin
- added J2: MSTBA8, Connector_Phoenix_MSTB:PhoenixContact_MSTBA_2,5_8-G-5,08_1x08_P5.08mm_Horizontal, symbol Connector_Generic:Conn_01x08
- added L1, L2: 330uH, loadbank:IND_HCTI-220-5.8, symbol Device:L
- added R1, R2, R3, R4: R, symbol Device:R
- added U1: LM2576HVT-5, Package_TO_SOT_THT:TO-220-5_P3.4x3.7mm_StaggerOdd_Lead3.8mm_Vertical, symbol Regulator_Switching:LM2576HVT-5
Connections:
- new net: F2.1, J2.7 (Pin_7)
- new net: C8.1, R1.2
- new net: C6.1, CR1.6 (BOOT), R4.2
- new net: F1.1, J2.3 (Pin_3)
- new net: C9.2, CR1.2 (SS_INH), D2.1 (K)
- new net: CR1.8 (FB), R1.1
- new net: D1.1 (K), L1.1, U1.2 (OUT)
- new net: C5.1, CR1.7 (COMP)
- new net +12V: C1.1, C2.1, J2.5 (Pin_5), U1.1 (VIN)
- new net +46V: C11.1, C7.1, J2.1 (Pin_1), R4.1
- new net +5V: C3.1, C4.1, F2.2, L1.2, U1.4 (FB)
- new net 12V(2): F1.2
- new net GND: C1.2, C2.2, C3.2, C4.2, D1.2 (A), HS1.1, J2.6 (Pin_6), J2.8 (Pin_8), U1.3 (GND), U1.5 (~{ON}/OFF)
- new net GND(2): HS1.2
- new net GND2: C11.2, C5.2, C6.2, C7.2, C8.2, C9.1, CR1.1 (GND), J2.2 (Pin_2), J2.4 (Pin_4)
Other:
- note added: "12V - 5V Regulator"
- note added: "46V - 12V Regulator"
