File: Hardware/High Current Board/High-Current/_autosave-High Current Board.kicad_pcb (KiCad board)
At the start: 2 copper layers, 174.3 x 152.3 mm, 37 parts, among them J1 8P8C_Shielded, J2 Conn_01x04, J3 GND, J4 Load Resistors Return, J5 +46V from Fuel Cell, K1 G2RL-1A-E, K2 G2RL-1A-E, Q1 NMOS_Substrate, Q2 NMOS, U1 TC4421AVAT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

Commit message: PCB Update for the schematic
Parts:
- moved F2 2.17 mm to (96.7, 152.3)
- moved F3 2.17 mm to (96.9, 161.2)
Routing:
- net /FUEL_CELL_CURRENT: track 18.6 -> 34.5 mm, vias 0 -> 1
- net /GATE_SIG: track 171.2 -> 156.1 mm, vias 0 -> 1
- net /3.3V: track 19.5 -> 33.2 mm, vias 0 -> 1
- net Net-(J2-Pin_4): track 21.6 -> 19.9 mm
- net /AIR_STARVE_RELAY: track 129.5 -> 128.2 mm, vias 0 -> 1
Other:
- board size 174.3 x 152.3 mm -> 174.3 x 151.9 mm
