File: Hardware/High Current Board/High-Current/High Current Board.kicad_pcb (KiCad board)
At the start: 2 copper layers, 174.3 x 152.3 mm, 37 parts, among them J1 8P8C_Shielded, J2 Conn_01x04, J3 GND, J4 Load Resistors Return, J5 +46V from Fuel Cell, K1 G2RL-1A-E, K2 G2RL-1A-E, Q1 NMOS_Substrate, Q2 NMOS, U1 TC4421AVAT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

Commit message: final update
Parts:
- moved J3 23.6 mm to (197.5, 161.2), turned to 180 degrees
- moved F2 2.17 mm to (96.7, 152.3)
- moved F3 2.17 mm to (96.9, 161.2)
Connections:
- J4 pad 1: (no net) -> Net-(J4-Pin_1)
Routing:
- net Net-(D2-A): track 214.7 -> 237.2 mm
- net /FUEL_CELL_CURRENT: track 18.6 -> 34.5 mm, vias 0 -> 1
- net /GATE_SIG: track 171.2 -> 155.4 mm, vias 0 -> 1
- net Net-(D1-A): track 19.7 -> 35.3 mm, vias 0 -> 2
- net /3.3V: track 19.5 -> 33.2 mm, vias 0 -> 1
- net GND: track 0.00 -> 2.00 mm, vias 0 -> 1
- net Net-(J2-Pin_4): track 21.6 -> 19.9 mm
- net /AIR_STARVE_RELAY: track 129.5 -> 128.2 mm, vias 0 -> 1
- added copper zone on B.Cu, net GND
- added copper zone on F.Cu, net GND
Other:
- board size 174.3 x 152.3 mm -> 174.3 x 151.9 mm
- board text added: "+46V AND LOAD RES (+)"
- board text added: "12V IN"
- board text added: "15A"
- board text added: "46V OUT"
- board text added: "5A"
- board text added: "GND"
- board text added: "High Current Board REV: 0.0"
- board text added: "LOAD RES (-)"
- board text added: "Only +46V wire should pass through current sensor loop"
- board text added: "RES (+)"
- board text added: "RES (-)"
- board text added: "TO CONTROLLER BOARD"
