File: Hardware/High Current Board/High-Current/High Current Board.kicad_pcb (KiCad board)
At the start: 2 copper layers, 174.3 x 151.9 mm, 37 parts, among them J1 8P8C_Shielded, J2 Conn_01x04, J3 GND, J4 Load Resistors Return, J5 +46V from Fuel Cell, K1 G2RL-1A-E, K2 G2RL-1A-E, Q1 NMOS_Substrate, Q2 NMOS, U1 TC4421AVAT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

Commit message: PCB Update - HC
Parts:
- removed Q2: NMOS, KiCADv6:SOT-227B
- added U2: ~, KiCADv6:GENESIC_MBR200100CTS, F.Cu at (167.8, 51.8)
Connections:
- R2 pad 1: Net-(Q2-D) -> GATE_DRIVE
Routing:
- net Net-(Q2-D): track 120.8 -> 0.00 mm
- net GATE_DRIVE: track 0.00 -> 116.2 mm
- net Net-(D2-A): track 237.2 -> 235.6 mm
Other:
- board size 174.3 x 151.9 mm -> 174.9 x 151.1 mm

Commit message: PCB Update 1.0
Needs a Revision Check and we good
Parts:
- moved D1 13.3 mm to (65.2, 110.4), turned to 90 degrees
- moved H1 12.6 mm to (228.0, 18.0)
- moved H4 12.6 mm to (228.0, 161.2)
- moved J1 12.2 mm to (132.5, 153.0)
- moved J2 12.2 mm to (71.2, 151.2)
- moved C1 12.2 mm to (143.8, 156.6)
- moved C10 12.2 mm to (216.0, 117.2)
- moved C11 12.2 mm to (216.0, 136.5)
- moved C12 12.2 mm to (172.8, 78.8)
- moved C13 12.2 mm to (109.2, 131.5)
- moved C2 12.2 mm to (143.8, 150.0)
- moved C3 12.2 mm to (147.6, 150.1)
- moved C4 12.2 mm to (73.7, 87.5)
- moved C5 12.2 mm to (73.7, 83.8)
- moved C6 12.2 mm to (215.0, 42.6)
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Routing:
- net Net-(D1-A): track 35.3 -> 24.4 mm
- net /AIR_STARVE_RELAY: track 128.2 -> 133.1 mm
- net +12V: track 109.8 -> 111.6 mm
- net /GATE_SIG: track 155.4 -> 155.9 mm

Commit message: Text update
Routing:
- net (no net): track 0.00 -> 0.71 mm
Changed lines of the file:
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@@
     (date "2024-01-11")
     (rev "0.0")
-    (comment 1 "University of Alberta EcoCar Team")
-    (comment 2 "Automated Resistive Load Bank Project")
+    (company "University of Alberta EcoCar Team")
+    (comment 1 "Automated Resistive Load Bank Project")
+    (comment 6 " ")
   )
   (layers
@@
     (effects (font (size 1.5 1.5) (thickness 0.3) bold) (justify left bottom))
   )
+  (segment (start 196 159.25) (end 195.5 158.75) (width 0.2) (layer "B.Cu") (net 0))
   (segment (start 149.116 154.25) (end 149.066 154.2) (width 0.2) (layer "F.Cu") (net 1))
   (segment (start 139.85 155.6) (end 139 154.75) (width 0.2) (layer "F.Cu") (net 1))
