File: Hardware/High Current Board/High-Current/High Current Board.kicad_sch (KiCad schematic)
At the start: 35 parts, among them J1 8P8C_Shielded, J2 Conn_01x04, J3 GND, J4 Load Resistors Return, J5 +46V from Fuel Cell, K1 G2RL-1A-E, K2 G2RL-1A-E, Q1 NMOS_Substrate, Q2 NMOS, U1 HO25-NPxSP33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

Commit message: Updated Schematic
Parts:
- removed C1, C3: 47nF, symbol Device:C
- removed C12, C13: C_Small, symbol Device:C_Small
- removed C2: 4.7nF, symbol Device:C
- removed C4: 01.uF, symbol Device:C
- removed C5: 10uF, symbol Device:C_Polarized_US
- removed L1, L2, L3, L4: L, symbol Device:L
- removed R1: 20k, symbol Device:R
- removed U1: HO25-NPxSP33, Sensor_Current:LEM_HO8-NP, symbol Sensor_Current:HO25-NPxSP33
- removed U2: TC4421, Package_DIP:DIP-8-N6_W7.62mm, symbol Driver_FET:TC4421
- added C1, C3: 47nF, Capacitor_SMD:C_0805_2012Metric, symbol Device:C_Small
- added C12, C13: 60uF, C4A-060_KEM, symbol 2024-01-06_11-24-14:C4ATDBW5600A30J
- added C2: 4.7nF, Capacitor_SMD:C_0805_2012Metric, symbol Device:C_Small
- added C4: 10uF, Capacitor_SMD:C_0201_0603Metric, symbol Device:C_Polarized_US
- added C5: 0.1uF, Capacitor_SMD:C_0805_2012Metric, symbol Device:C
- added L1, L5: L_Coupled, KiCADv6:FIL_CMX1616Z171B-10, symbol Device:L_Coupled
- added R3: 20k, Resistor_SMD:R_2512_6332Metric_Pad1.40x3.35mm_HandSolder, symbol Device:R
- added U1: TC4421AVAT, TC4421AVAT:TO170P1066X482X1572-5, symbol TC4421AVAT:TC4421AVAT
- added U3: HO 25-P, HO 25-P_LEM, symbol HO25-P Current Sensor:HO_25-P
- C10, C11, C6, C7, C8, C9: footprint (none) -> Capacitor_THT:CP_Radial_D10.0mm_P3.50mm
- D2: footprint (none) -> Diode_SMD:D_3220_8050Metric
- F1: footprint (none) -> Fuse:Fuse_1206_3216Metric
- F2, F3: footprint (none) -> Fuse:Fuseholder_Blade_Mini_Keystone_3568
- J1: footprint (none) -> Connector_RJ:RJ45_Amphenol_RJHSE538X
- J2: footprint (none) -> Connector_Phoenix_MSTB:PhoenixContact_MSTBA_2,5_4-G-5,08_1x04_P5.08mm_Horizontal
- J3, J4, J5: footprint (none) -> Connector_Wuerth:Wuerth_WR-WTB_64801011622_1x10_P1.50mm_Vertical
- Q1: footprint (none) -> KiCADv6:SOT65P210X100-3N
- Q2: footprint (none) -> KiCADv6:SOT-227B
- R2: footprint (none) -> Resistor_SMD:R_2512_6332Metric_Pad1.40x3.35mm_HandSolder
Connections:
- net +12V: now also C4.2, C5.1, U1.3 (VDD)
- net 3.3V: now also C1.1, R3.1, U3.1 (+UC)
- net 3.3V_RETURN: now also C1.2, C2.1, C3.1, C3.2, R3.2, U3.2 (0V), U3.4 (VREF), U3.5 (OCD)
- net FUEL_CELL_CURRENT: now also C2.2, U3.3 (VOUT)
- net GATE_SIG: now also U1.1 (VIN)
- net GND: now also C12.1, C12.2, C13.1, C13.2, C4.1, C5.2, U1.2 (GND), U1.4 (GND__1)
- net at J4.1 (Pin_1): now also L1.1, L1.3, L5.1, L5.3
- net at D2.2 (A), Q2.1 (D): now also L1.2, L1.4, L5.2, L5.4
- net at R2.2: now also U1.5 (OUTPUT)
- net +48V renamed +46V
- net +46V: now also C12.3, C12.4, C13.3, C13.4
Other:
- note added: "From Voltage Regulator Board"
- note added: "To Voltage Regulator Board"
- note added: "resistor"
- note removed: "NEED 46 THO"
- note removed: "VDD=3*2?"
- note removed: "film capacitors"
- note removed: "need 46"
- moved on the sheet: D1, D2, F1, F2, F3, J1, J2, K1, K2, Q1, Q2, R2

Commit message: PCB Update for the schematic
Parts:
- added H1, H2, H3, H4: MountingHole, MountingHole:MountingHole_2.7mm_M2.5, symbol Mechanical:MountingHole
- C10, C11, C6, C7, C8, C9: footprint Capacitor_THT:CP_Radial_D10.0mm_P3.50mm -> Capacitor_THT:CP_Radial_D16.0mm_P7.50mm
- D1: footprint (none) -> Diode_SMD:D_3220_8050Metric
- U1: footprint TC4421AVAT:TO170P1066X482X1572-5 -> KiCADv6:TO170P1066X482X1572-5
Connections:
- net AIR_STARVE_RELAYS is gone; now on net AIR_STARVE_RESISTORS: J2.2 (Pin_2)
- net 3.3V_RETURN: no longer C3.2, U3.4 (VREF)
- new net: C3.2, U3.4 (VREF)
Other:
- note added: "Mounting Holes (M2.5)"
- moved on the sheet: D1, K1, K2, Q1

Commit message: PCB Update - HC
Parts:
- Q2: footprint KiCADv6:SOT-227B -> filmcapacitorsfootprint:SOT-23_MCC
Connections:
- net at J4.1 (Pin_1), L5.1, L5.3: now also L1.2, L1.4; no longer L1.1, L1.3
- net at D2.2 (A), L5.2, L5.4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: now also L1.1, L1.3; no longer L1.2, L1.4
Other:
- moved on the sheet: L1
Changed lines of the file:
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@@
   (junction (at 118.11 113.03) (diameter 0) (color 0 0 0 0)
   )
+  (wire (pts (xy 95.25 134.62) (xy 105.41 134.62))
+    (stroke (width 0) (type default))
+  )
   (wire (pts (xy 237.49 111.76) (xy 256.54 111.76))
     (stroke (width 0) (type default))
@@
   )
   (wire (pts (xy 138.43 90.17) (xy 138.43 92.71))
-    (stroke (width 0) (type default))
-  )
-  (wire (pts (xy 105.41 134.62) (xy 95.25 134.62))
     (stroke (width 0) (type default))
   )
@@
       (effects (font (size 1.27 1.27)) (justify left) hide)
     )
-    (property "Footprint" "KiCADv6:SOT-227B" (at 85.09 132.08 0)
+    (property "Footprint" "filmcapacitorsfootprint:SOT-23_MCC" (at 85.09 132.08 0)
       (effects (font (size 1.27 1.27)) hide)
     )
@@
     )
   )
-  (symbol (lib_id "Device:L_Coupled") (at 78.74 125.73 0) (unit 1)
-    (in_bom yes) (on_board yes) (dnp no)
-    (property "Reference" "L1" (at 78.74 121.92 0)
-      (effects (font (size 1.27 1.27)))
-    )
-    (property "Value" "L_Coupled" (at 78.359 120.65 0)
-      (effects (font (size 1.27 1.27)) hide)
-    )
+  (symbol (lib_id "Device:L_Coupled") (at 78.74 125.73 180) (unit 1)
+    (in_bom yes) (on_board yes) (dnp no)
+    (property "Reference" "L1" (at 78.74 129.54 0)
+      (effects (font (size 1.27 1.27)))
+    )
+    (property "Value" "L_Coupled" (at 79.121 130.81 0)
+      (effects (font (size 1.27 1.27)) hide)
+    )

Commit message: PCB Update 1.0
Needs a Revision Check and we good
Parts:
- removed Q2: NMOS, filmcapacitorsfootprint:SOT-23_MCC, symbol Simulation_SPICE:NMOS
- added U2: ~, KiCADv6:GENESIC_MBR200100CTS, symbol Extra Symbols:SOT-227
Connections:
- net GND: now also U2.1 (S), U2.3 (S)
- net at D2.2 (A), L1.1, L1.3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: now also U2.4 (D)
- net at R2.1: now also U2.2 (G)
Other:
- moved on the sheet: D2
